File: SB_PCB_MEDAL/SB_PCB_MEDAL.sch (EAGLE design)
At the start: 9 parts, among them IC1 ATTINY44A-SSU

Commit message: modified connections to button cell and added text for the ICSP header to the PCB
Connections:
- removed net N$2: BT1.+
- net GND: now also IC1.GND
- net VCC: now also BT1.+
Changed lines of the file:
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@@
 Anton Nikitin - Henry Oliver-Edwards</text>
 <text x="-20.32" y="66.04" size="1.778" layer="97">VCC</text>
+<text x="91.44" y="66.04" size="1.778" layer="97">GND</text>
+<text x="50.8" y="27.94" size="1.778" layer="97">VCC</text>
 </plain>
 <instances>
@@
 <pinref part="GND2" gate="1" pin="GND"/>
 </segment>
+<segment>
+<pinref part="IC1" gate="G$1" pin="GND"/>
+<wire x1="88.9" y1="66.04" x2="91.44" y2="66.04" width="0.1524" layer="91"/>
+</segment>
 </net>
 <net name="VCC" class="0">
+<segment>
+<pinref part="IC1" gate="G$1" pin="VCC"/>
+<wire x1="-7.62" y1="66.04" x2="-20.32" y2="66.04" width="0.1524" layer="91"/>
+</segment>
 <segment>
 <pinref part="ICSP" gate="1" pin="5"/>
@@
 </segment>
 <segment>
-<pinref part="IC1" gate="G$1" pin="VCC"/>
-<wire x1="-7.62" y1="66.04" x2="-20.32" y2="66.04" width="0.1524" layer="91"/>
-</segment>
-</net>
-<net name="N$2" class="0">
-<segment>
 <pinref part="BT1" gate="G$1" pin="+"/>
