File: SB_PCB_MEDAL/SB_PCB_MEDAL.sch (EAGLE design)
At the start: 40 parts, among them U1 ATMEGA16U2-AU, X1 MINI-USB_SHIELD5P2-32005-601, Y1 FOXSDLF_120-20

Commit message: modify board
Parts:
- added C1, C2, C3, C4: MC0805B104K250CT, SamacSys_Parts:MC0805B104K250CT
- added R7, R8: 22 Ω, resistor:R-EU_M0805
- added R9: (no value), rcl:R-EU_0204/7
- added S1: 1825910-6, SamacSys_Parts:1825910-6
Connections:
- removed net PA0: R1.1
- removed net PA1: R2.1
- removed net PA2: R3.1
- removed net PA3: R4.1
- removed net PB0: R5.1
- removed net PB1: R6.1
- new net D+: R8.1, X1G41.3
- new net D-: R7.1, X1G41.2
- new net N$10: R9.2, S1.2
- new net N$11: C3.1, U1.AVCC
- new net N$14: R8.2, U1.D+
- new net N$15: R7.2, U1.D-
- new net N$17: X1G41.4
- new net N$20: U1.(RTS_/_AIN5_/_INT6)_PD6
- new net N$21: U1./_HWB_/_AIN6_/_T0_/_INT7)_PD7
- new net N$9: C1.1, U1.VCC
- new net PD0: R1.1, U1.(OC.0B_/_INT0)_PD0
- new net PD1: R2.1, U1.(AIN0_/_INT1)_PD1
- new net PD2: R3.1, U1.(RXD1_/_AIN1_/_INT2)_PD2
- new net PD3: R4.1, U1.(TXD1_/_INT3)_PD3
- new net PD4: R5.1, U1.(INT5/_AIN3)_PD4
- new net PD5: R6.1, U1.(XCK_AIN4_/_PCINT12)_PD5
- new net RESET: S1.1
- new net UGND: U1.UGND, X1G41.5
- new net UVCC: C2.1, U1.UVCC
- new net VOUT_REG: R9.1
- new net XTAL1: U1.XTAL1
- new net XTAL2: U1.(PC0)_XTAL2
- net GND: now also C4.1, S1.3, S1.4, U1.GND
- net VCC: now also C1.2, C2.2, C3.2, C4.2, U1.UCAP, X1G41.1
Other:
- note added: "Active Low Reset"
- note added: "D+"
- note added: "D-"
- note added: "ID"
- note added: "UNUSED"
- note removed: "PA0"
- note removed: "PA1"
- note removed: "PA2"
- note removed: "PA3"
- note removed: "PB0"
- note removed: "PB1"
- moved on the sheet: ICSP, U1, X1, Y1
