File: SB_PCB_MEDAL/SB_PCB_MEDAL.brd (EAGLE design)
At the start: 90 x 90 mm, 40 parts, among them U1 ATMEGA16U2-AU, Y1 FOXSDLF_120-20

Commit message: modify board
Parts:
- added C1, C2, C3: (no value), SamacSys_Parts:CAPC2012X60N
- added C4: MC0805B104K250CT, SamacSys_Parts:CAPC2012X60N
- added R7, R8: 22 Ω, resistor:M0805
- added R9: (no value), rcl:0204/7
- added S1: 1825910-6, SamacSys_Parts:1825910-6
- moved Y1 6.00 mm to (24.0, 6.00)
Connections:
- removed net AVCC: U1.32
- removed net PA0: R1.1
- removed net PA1: R2.1
- removed net PA2: R3.1
- removed net PA3: R4.1
- removed net PB0: R5.1
- removed net PB1: R6.1
- new net D+: R8.1, X1.3
- new net D-: R7.1, X1.2
- new net N$10: R9.2, S1.2
- new net N$11: C3.1, U1.32
- new net N$14: R8.2, U1.29
- new net N$15: R7.2, U1.30
- new net N$17: X1.4
- new net N$20: U1.12
- new net N$21: U1.13
- new net N$9: C1.1, U1.4
- new net PD0: R1.1, U1.6
- new net PD1: R2.1, U1.7
- new net PD2: R3.1, U1.8
- new net PD3: R4.1, U1.9
- new net PD4: R5.1, U1.10
- new net PD5: R6.1, U1.11
- new net RESET: S1.1
- new net UGND: U1.28, X1.5
- new net VOUT_REG: R9.1
- new net XTAL1: U1.1
- new net XTAL2: U1.2
- net GND: now also C4.1, S1.3, S1.4, U1.3
- net UVCC: now also C2.1
- net VCC: now also C1.2, C2.2, C3.2, C4.2, U1.27, X1.1; no longer U1.4
